Commit message: Organise URDF

File: auldbot_description/urdf/auldbot.urdf.xacro (robot description, xacro)
@@ -1,11 +1,11 @@
-<?xml version="1.0" ?>
+<?xml version="1.0"?>
 <robot name="auldbot" xmlns:xacro="http://www.ros.org/wiki/xacro">
   <!-- ===================== HARDWARE PARAMETERS ===================== -->
-  <xacro:arg name="serial_port" default="/dev/auldbot_servos" />
-  <xacro:arg name="baud_rate" default="1000000" />
-  <xacro:arg name="left_wheel_id" default="7" />
-  <xacro:arg name="right_wheel_id" default="9" />
-  <xacro:arg name="velocity_scale" default="2744.0" />
-  <xacro:arg name="acceleration" default="0" />
+  <xacro:arg name="serial_port"    default="/dev/auldbot_servos"/>
+  <xacro:arg name="baud_rate"      default="1000000"/>
+  <xacro:arg name="left_wheel_id"  default="7"/>
+  <xacro:arg name="right_wheel_id" default="9"/>
+  <xacro:arg name="velocity_scale" default="2744.0"/>
+  <xacro:arg name="acceleration"   default="0"/>
   <!-- ===================== MEASUREMENTS ===================== -->
   <!--
@@ -14,194 +14,156 @@
   -->
   <!-- Heights above ground -->
-  <xacro:property name="base_plate_top_height" value="0.016" />
-  <xacro:property name="lidar_ground_height" value="0.054" />
-  <xacro:property name="cam_ground_height" value="0.094" />
+  <xacro:property name="base_plate_top_height" value="0.016"/>
+  <xacro:property name="lidar_ground_height"   value="0.054"/>
+  <xacro:property name="cam_ground_height"     value="0.094"/>
   <!-- Plate geometry -->
-  <xacro:property name="chassis_radius" value="0.115" />
-  <xacro:property name="plate_thickness" value="0.006" />
-  <xacro:property name="plate_gap" value="0.050" />
-  <xacro:property name="plate_mass" value="0.01" />  <!-- dummy -->
+  <xacro:property name="chassis_radius"  value="0.115"/>
+  <xacro:property name="plate_thickness" value="0.006"/>
+  <xacro:property name="plate_gap"       value="0.050"/>
+  <xacro:property name="plate_mass"      value="0.01"/>  <!-- dummy -->
   <!-- Drive wheels (STS3215) -->
-  <xacro:property name="wheel_radius" value="0.028" />
-  <xacro:property name="wheel_width" value="0.006" />
-  <xacro:property name="wheel_mass" value="0.05" />  <!-- dummy -->
-  <xacro:property name="wheel_separation" value="0.219" />
+  <xacro:property name="wheel_radius"     value="0.0325"/>
+  <xacro:property name="wheel_width"      value="0.006"/>
+  <xacro:property name="wheel_mass"       value="0.05"/>  <!-- dummy -->
+  <xacro:property name="wheel_separation" value="0.219"/>
+  <xacro:property name="axle_z"           value="0.0095"/>
   <!-- Caster -->
-  <xacro:property name="caster_radius" value="0.006" />  <!-- assumed -->
-  <xacro:property name="caster_mass" value="0.01" />   <!-- dummy -->
-  <xacro:property name="caster_x" value="0.100" />  <!-- assumed -->
+  <xacro:property name="caster_radius" value="0.016"/>  <!-- assumed -->
+  <xacro:property name="caster_mass"   value="0.01"/>   <!-- dummy -->
+  <xacro:property name="caster_x"      value="0.100"/>  <!-- assumed -->
+  <xacro:property name="caster_z"      value="${-caster_radius/2}"/>  <!-- assumed -->
   <!-- Lidar -->
-  <xacro:property name="lidar_x" value="0.080" />
+  <xacro:property name="lidar_x" value="0.080"/>
+  <xacro:property name="lidar_z" value="0.038"/>
   <!-- Camera -->
-  <xacro:property name="cam_x" value="0.110" />
+  <xacro:property name="cam_x" value="0.110"/>
+  <xacro:property name="cam_z" value="0.021"/>
   <!-- ===================== DERIVED POSITIONS (base_link frame) ===================== -->
-  <xacro:property
-    name="base_plate_z"
-    value="${base_plate_top_height - plate_thickness / 2 - wheel_radius}"
-  />
-  <xacro:property
-    name="top_plate_z"
-    value="${base_plate_top_height + plate_gap + plate_thickness / 2 - wheel_radius}"
-  />
-  <xacro:property
-    name="lidar_z"
-    value="${lidar_ground_height - wheel_radius}"
-  />
-  <xacro:property name="cam_z" value="${cam_ground_height - wheel_radius}" />
+  <xacro:property name="base_plate_z" value="${-axle_z}"/>
+  <xacro:property name="top_plate_z"  value="${plate_gap + plate_thickness}"/>
+  <!-- ===================== Materials ===================== -->
+  <material name="black"><color rgba="0.1 0.1 0.1 1.0"/></material>
+  <material name="blue"><color rgba="0.0 0.471 0.749 1.0"/></material>
   <!-- ===================== LINKS ===================== -->
-  <link name="base_footprint" />
-  <link name="base_link" />
+  <link name="base_footprint"/>
+  <link name="base_link"/>
   <joint name="base_footprint_joint" type="fixed">
-    <parent link="base_footprint" />
-    <child link="base_link" />
-    <origin xyz="0 0 ${wheel_radius}" rpy="0 0 0" />
+    <parent link="base_footprint"/>
+    <child  link="base_link"/>
+    <origin xyz="0 0 ${wheel_radius}" rpy="0 0 0"/>
   </joint>
   <link name="base_plate_link">
     <visual>
-      <geometry><cylinder
-          radius="${chassis_radius}"
-          length="${plate_thickness}"
-        /></geometry>
+      <geometry><cylinder radius="${chassis_radius}" length="${plate_thickness}"/></geometry>
+      <material name="black"/>
     </visual>
     <collision>
-      <geometry><cylinder
-          radius="${chassis_radius}"
-          length="${plate_thickness}"
-        /></geometry>
+      <geometry><cylinder radius="${chassis_radius}" length="${plate_thickness}"/></geometry>
     </collision>
     <inertial>
-      <mass value="${plate_mass}" />
-      <inertia
-        ixx="0.000033"
-        ixy="0"
-        ixz="0"
-        iyy="0.000033"
-        iyz="0"
-        izz="0.000066"
-      />
+      <mass value="${plate_mass}"/>
+      <inertia ixx="0.000033" ixy="0" ixz="0"
+               iyy="0.000033" iyz="0"
+               izz="0.000066"/>
     </inertial>
   </link>
   <joint name="base_plate_joint" type="fixed">
-    <parent link="base_link" />
-    <child link="base_plate_link" />
-    <origin xyz="0 0 ${base_plate_z}" rpy="0 0 0" />
+    <parent link="base_link"/>
+    <child  link="base_plate_link"/>
+    <origin xyz="0 0 ${base_plate_z}" rpy="0 0 0"/>
   </joint>
   <link name="top_plate_link">
     <visual>
-      <geometry><cylinder
-          radius="${chassis_radius}"
-          length="${plate_thickness}"
-        /></geometry>
+      <geometry><cylinder radius="${chassis_radius}" length="${plate_thickness}"/></geometry>
+      <material name="black"/>
     </visual>
     <collision>
-      <geometry><cylinder
-          radius="${chassis_radius}"
-          length="${plate_thickness}"
-        /></geometry>
+      <geometry><cylinder radius="${chassis_radius}" length="${plate_thickness}"/></geometry>
     </collision>
     <inertial>
-      <mass value="${plate_mass}" />
-      <inertia
-        ixx="0.000033"
-        ixy="0"
-        ixz="0"
-        iyy="0.000033"
-        iyz="0"
-        izz="0.000066"
-      />
+      <mass value="${plate_mass}"/>
+      <inertia ixx="0.000033" ixy="0" ixz="0"
+               iyy="0.000033" iyz="0"
+               izz="0.000066"/>
     </inertial>
   </link>
   <joint name="top_plate_joint" type="fixed">
-    <parent link="base_link" />
-    <child link="top_plate_link" />
-    <origin xyz="0 0 ${top_plate_z}" rpy="0 0 0" />
+    <parent link="base_plate_link"/>
+    <child  link="top_plate_link"/>
+    <origin xyz="0 0 ${top_plate_z}" rpy="0 0 0"/>
   </joint>
   <xacro:macro name="wheel" params="name y_reflect">
     <link name="${name}_wheel_link">
       <visual>
-        <geometry><cylinder
-            radius="${wheel_radius}"
-            length="${wheel_width}"
-          /></geometry>
-        <origin xyz="0 0 0" rpy="${pi/2} 0 0" />
+        <geometry><cylinder radius="${wheel_radius}" length="${wheel_width}"/></geometry>
+        <origin xyz="0 0 0" rpy="${pi/2} 0 0"/>
       </visual>
       <collision>
-        <geometry><cylinder
-            radius="${wheel_radius}"
-            length="${wheel_width}"
-          /></geometry>
-        <origin xyz="0 0 0" rpy="${pi/2} 0 0" />
+        <geometry><cylinder radius="${wheel_radius}" length="${wheel_width}"/></geometry>
+        <origin xyz="0 0 0" rpy="${pi/2} 0 0"/>
       </collision>
       <inertial>
-        <mass value="${wheel_mass}" />
-        <inertia
-          ixx="0.000010"
-          ixy="0"
-          ixz="0"
-          iyy="0.000020"
-          iyz="0"
-          izz="0.000010"
-        />
+        <mass value="${wheel_mass}"/>
+        <inertia ixx="0.000010" ixy="0" ixz="0"
+                 iyy="0.000020" iyz="0"
+                 izz="0.000010"/>
       </inertial>
     </link>
     <joint name="${name}_wheel_joint" type="continuous">
-      <parent link="base_link" />
-      <child link="${name}_wheel_link" />
-      <origin xyz="0 ${y_reflect * wheel_separation / 2} 0" rpy="0 0 0" />
-      <axis xyz="0 1 0" />
+      <parent link="base_link"/>
+      <child  link="${name}_wheel_link"/>
+      <origin xyz="0 ${y_reflect * wheel_separation / 2} 0" rpy="0 0 0"/>
+      <axis xyz="0 1 0"/>
     </joint>
   </xacro:macro>
-  <xacro:wheel name="left" y_reflect=" 1" />
-  <xacro:wheel name="right" y_reflect="-1" />
+  <xacro:wheel name="left"  y_reflect=" 1"/>
+  <xacro:wheel name="right" y_reflect="-1"/>
   <link name="caster_link">
     <visual>
-      <geometry><sphere radius="${caster_radius}" /></geometry>
+      <geometry><sphere radius="${caster_radius}"/></geometry>
     </visual>
     <collision>
-      <geometry><sphere radius="${caster_radius}" /></geometry>
+      <geometry><sphere radius="${caster_radius}"/></geometry>
     </collision>
     <inertial>
-      <mass value="${caster_mass}" />
+      <mass value="${caster_mass}"/>
       <!-- dummy inertia -->
-      <inertia
-        ixx="0.000001"
-        ixy="0"
-        ixz="0"
-        iyy="0.000001"
-        iyz="0"
-        izz="0.000001"
-      />
+      <inertia ixx="0.000001" ixy="0" ixz="0"
+               iyy="0.000001" iyz="0"
+               izz="0.000001"/>
     </inertial>
   </link>
   <joint name="caster_joint" type="fixed">
-    <parent link="base_link" />
-    <child link="caster_link" />
-    <origin xyz="${caster_x} 0 ${caster_radius - wheel_radius}" rpy="0 0 0" />
+    <parent link="base_plate_link"/>
+    <child  link="caster_link"/>
+    <origin xyz="${caster_x} 0 ${caster_z}" rpy="0 0 0"/>
   </joint>
   <link name="lidar_link">
     <visual>
-      <geometry><cylinder radius="0.038" length="0.04" /></geometry>
+      <geometry><cylinder radius="0.038" length="0.04"/></geometry>
+      <material name="blue"/>
     </visual>
   </link>
   <joint name="lidar_joint" type="fixed">
-    <parent link="base_link" />
-    <child link="lidar_link" />
-    <origin xyz="${lidar_x} 0 ${lidar_z}" rpy="0 0 ${pi/2}" />
+    <parent link="base_plate_link"/>
+    <child  link="lidar_link"/>
+    <origin xyz="${lidar_x} 0 ${lidar_z}" rpy="0 0 ${pi/2}"/>
   </joint>
   <link name="camera_link">
     <visual>
-      <geometry><box size="0.025 0.025 0.025" /></geometry>
+      <geometry><box size="0.025 0.025 0.025"/></geometry>
+      <material name="blue"/>
     </visual>
   </link>
   <joint name="camera_joint" type="fixed">
-    <parent link="base_link" />
-    <child link="camera_link" />
-    <origin xyz="${cam_x} 0 ${cam_z}" rpy="0 0 0" />
+    <parent link="top_plate_link"/>
+    <child  link="camera_link"/>
+    <origin xyz="${cam_x} 0 ${cam_z}" rpy="0 0 0"/>
   </joint>
-  <link name="camera_optical_link" />
+  <link name="camera_optical_link"/>
   <joint name="camera_optical_joint" type="fixed">
-    <parent link="camera_link" />
-    <child link="camera_optical_link" />
-    <origin xyz="0 0 0" rpy="${-pi/2} 0 ${-pi/2}" />
+    <parent link="camera_link"/>
+    <child  link="camera_optical_link"/>
+    <origin xyz="0 0 0" rpy="${-pi/2} 0 ${-pi/2}"/>
   </joint>
   <!-- ===================== ROS2 CONTROL ===================== -->
@@ -217,12 +179,12 @@
     </hardware>
     <joint name="left_wheel_joint">
-      <command_interface name="velocity" />
-      <state_interface name="velocity" />
-      <state_interface name="position" />
+      <command_interface name="velocity"/>
+      <state_interface   name="velocity"/>
+      <state_interface   name="position"/>
     </joint>
     <joint name="right_wheel_joint">
-      <command_interface name="velocity" />
-      <state_interface name="velocity" />
-      <state_interface name="position" />
+      <command_interface name="velocity"/>
+      <state_interface   name="velocity"/>
+      <state_interface   name="position"/>
     </joint>
   </ros2_control>

Commit message: fix: lidar was rotateed by 180 degrees

File: auldbot_description/urdf/auldbot.urdf.xacro (robot description, xacro)
@@ -150,4 +150,11 @@
     <origin xyz="${lidar_x} 0 ${lidar_z}" rpy="0 0 ${pi/2}"/>
   </joint>
+  <!-- Scan frame can be rotated independently from physical lidar mounting -->
+  <link name="lidar_scan_link"/>
+  <joint name="lidar_scan_joint" type="fixed">
+    <parent link="lidar_link"/>
+    <child  link="lidar_scan_link"/>
+    <origin xyz="0 0 0" rpy="0 0 ${pi}"/>
+  </joint>
   <link name="camera_link">
     <visual>

Commit message: fix: measured and corrected all calibrations

File: auldbot_description/urdf/auldbot.urdf.xacro (robot description, xacro)
@@ -6,5 +6,5 @@
   <xacro:arg name="left_wheel_id"  default="7"/>
   <xacro:arg name="right_wheel_id" default="9"/>
-  <xacro:arg name="velocity_scale" default="2744.0"/>
+  <xacro:arg name="velocity_scale" default="674.1"/>
   <xacro:arg name="acceleration"   default="0"/>
   <!-- ===================== MEASUREMENTS ===================== -->
@@ -26,5 +26,5 @@
   <xacro:property name="wheel_width"      value="0.006"/>
   <xacro:property name="wheel_mass"       value="0.05"/>  <!-- dummy -->
-  <xacro:property name="wheel_separation" value="0.219"/>
+  <xacro:property name="wheel_separation" value="0.217"/>
   <xacro:property name="axle_z"           value="0.0095"/>
   <!-- Caster -->

Commit message: feat: moved to dwb for planning

File: auldbot_description/urdf/auldbot.urdf.xacro (robot description, xacro)
@@ -26,5 +26,5 @@
   <xacro:property name="wheel_width"      value="0.006"/>
   <xacro:property name="wheel_mass"       value="0.05"/>  <!-- dummy -->
-  <xacro:property name="wheel_separation" value="0.217"/>
+  <xacro:property name="wheel_separation" value="0.22"/>
   <xacro:property name="axle_z"           value="0.0095"/>
   <!-- Caster -->
