Commit message: Add use_sim branch to URDF: gz_ros2_control + simulated lidar
With use_sim:=true the ros2_control hardware plugin swaps from
MoteHardware to gz_ros2_control/GazeboSimSystem, the gz_ros2_control
system plugin is attached (controller params file passed via the
sim_controllers_file arg), the fixed caster becomes frictionless, and a
gpu_lidar matching the RPLIDAR C1 (specs added to robot.yaml under
lidar.sim) publishes in lidar_scan_link like the real driver.

Without the flag the xacro output is byte-identical to before, and the
sim output converts cleanly with 'gz sdf -p'.

Co-Authored-By: Claude Fable 5 <noreply@anthropic.com>

File: mote_description/urdf/mote.urdf.xacro (robot description, xacro)
@@ -2,4 +2,10 @@
 <robot name="mote" xmlns:xacro="http://www.ros.org/wiki/xacro">
   <xacro:property name="cfg" value="${xacro.load_yaml('$(find mote_description)/config/robot.yaml')}"/>
+  <!-- Simulation: swaps MoteHardware for gz_ros2_control and adds gz sensors.
+       sim_controllers_file is the controller params file gz_ros2_control loads
+       (sim_launch.py generates it, injecting wheel geometry from this yaml). -->
+  <xacro:arg name="use_sim" default="false"/>
+  <xacro:arg name="sim_controllers_file" default=""/>
+  <xacro:property name="use_sim" value="$(arg use_sim)"/>
   <!-- ===================== MEASUREMENTS ===================== -->
   <!--
@@ -170,4 +176,5 @@
   <!-- ===================== ROS2 CONTROL ===================== -->
   <ros2_control name="mote_hardware" type="system">
+    <xacro:unless value="${use_sim}">
     <hardware>
       <plugin>mote_hardware/MoteHardware</plugin>
@@ -179,4 +186,10 @@
       <param name="acceleration">${cfg['servos']['acceleration']}</param>
     </hardware>
+    </xacro:unless>
+    <xacro:if value="${use_sim}">
+    <hardware>
+      <plugin>gz_ros2_control/GazeboSimSystem</plugin>
+    </hardware>
+    </xacro:if>
     <joint name="left_wheel_joint">
       <command_interface name="velocity"/>
@@ -190,3 +203,44 @@
     </joint>
   </ros2_control>
+  <xacro:if value="${use_sim}">
+    <!-- ===================== SIMULATION (Gazebo) ===================== -->
+    <gazebo>
+      <plugin filename="gz_ros2_control-system"
+              name="gz_ros2_control::GazeboSimROS2ControlPlugin">
+        <parameters>$(arg sim_controllers_file)</parameters>
+      </plugin>
+    </gazebo>
+    <!-- Caster is a fixed sphere: frictionless so it slides instead of dragging -->
+    <gazebo reference="caster_link">
+      <mu1>0.0</mu1>
+      <mu2>0.0</mu2>
+    </gazebo>
+    <xacro:property name="lidar_sim" value="${cfg['lidar']['sim']}"/>
+    <gazebo reference="lidar_link">
+      <sensor name="lidar" type="gpu_lidar">
+        <!-- Rotated to match lidar_scan_link so data agrees with the frame_id -->
+        <pose>0 0 0 0 0 ${pi}</pose>
+        <topic>scan</topic>
+        <gz_frame_id>lidar_scan_link</gz_frame_id>
+        <update_rate>${lidar_sim['update_rate']}</update_rate>
+        <always_on>true</always_on>
+        <visualize>false</visualize>
+        <lidar>
+          <scan>
+            <horizontal>
+              <samples>${lidar_sim['samples']}</samples>
+              <resolution>1</resolution>
+              <min_angle>${-pi}</min_angle>
+              <max_angle>${pi}</max_angle>
+            </horizontal>
+          </scan>
+          <range>
+            <min>${lidar_sim['range_min']}</min>
+            <max>${lidar_sim['range_max']}</max>
+            <resolution>0.01</resolution>
+          </range>
+        </lidar>
+      </sensor>
+    </gazebo>
+  </xacro:if>
 </robot>

Commit message: Misc cleanups: rviz display, caster height, rename clean task
- mote.rviz: show the SLAM pose graph, tune laser intensity range and
  the default top-down view scale
- URDF: derive caster_z from wheel_radius/axle_z so the caster sits at
  the true ground-contact height instead of a guessed offset
- pixi: rename the `clean` task to `kill` (it kills stale ROS processes);
  update the CLAUDE.md reference to match

Co-Authored-By: Claude Opus 4.8 <noreply@anthropic.com>
Claude-Session: https://claude.ai/code/session_01QXgJsGhCMsQ2yf4js6dDqo

File: mote_description/urdf/mote.urdf.xacro (robot description, xacro)
@@ -32,5 +32,5 @@
   <xacro:property name="caster_mass"   value="0.01"/>   <!-- dummy -->
   <xacro:property name="caster_x"      value="0.100"/>  <!-- assumed -->
-  <xacro:property name="caster_z"      value="${-caster_radius/2}"/>  <!-- assumed -->
+  <xacro:property name="caster_z"      value="${caster_radius - (wheel_radius - axle_z)}"/>
   <!-- Lidar -->
   <xacro:property name="lidar_x" value="0.080"/>

Commit message: Add a simulated RGB camera to the Gazebo sim
Add a gz camera sensor (use_sim branch only) that publishes /image_raw and
/camera_info in frame camera_optical_link, mirroring the simulated lidar, so
camera perception (L1) can be developed and tested headless. Sim params live in
robot.yaml's camera.sim block (FOV matched to the calibrated real lens);
sim_launch.py bridges the two topics; the sim smoke test now asserts /image_raw.
Non-sim URDF output is unchanged.

Co-Authored-By: Claude Opus 4.8 <noreply@anthropic.com>

File: mote_description/urdf/mote.urdf.xacro (robot description, xacro)
@@ -243,4 +243,29 @@
       </sensor>
     </gazebo>
+    <xacro:property name="camera_sim" value="${cfg['camera']['sim']}"/>
+    <gazebo reference="camera_link">
+      <sensor name="camera" type="camera">
+        <!-- gz_frame_id is the optical frame so the published image/camera_info
+             frame_id follows the ROS optical convention (z-forward). The sensor
+             body is camera_link (+X-forward), which gz uses as the view axis. -->
+        <topic>image_raw</topic>
+        <gz_frame_id>camera_optical_link</gz_frame_id>
+        <update_rate>${camera_sim['update_rate']}</update_rate>
+        <always_on>true</always_on>
+        <visualize>false</visualize>
+        <camera>
+          <horizontal_fov>${camera_sim['horizontal_fov']}</horizontal_fov>
+          <image>
+            <width>${camera_sim['width']}</width>
+            <height>${camera_sim['height']}</height>
+            <format>R8G8B8</format>
+          </image>
+          <clip>
+            <near>${camera_sim['near']}</near>
+            <far>${camera_sim['far']}</far>
+          </clip>
+        </camera>
+      </sensor>
+    </gazebo>
   </xacro:if>
 </robot>

Commit message: SO-101 follower arm bring-up: joint states + safe jog control
Bring the mounted SO-101 follower arm under software control: live joint
states, safe soft-limited joint commands, a jog CLI, and bench tools. There
is no leader arm and none is assumed anywhere.

Stack decision (documented in mote_arm/README.md): direct Feetech control,
not LeRobot. The arm servos are the same STS-class Feetech bus as the drive
wheels, so this reuses the servo approach rather than pulling torch onto the
lean Pi env (which the repo keeps torch off, isolating inference off-board).
The only new dep is the pure-Python feetech-servo-sdk (scservo_sdk).

New mote_arm package (Python/ament):
- config.py: parses robot.yaml `arm:`; encoder<->rad conversion + soft-limit
  clamping. ROS-free and unit-tested (15 tests) so the safety maths is
  verified without hardware.
- bus.py: FeetechBus, a thin scservo_sdk wrapper (lazy import so
  build/lint/test stay hardware-free); register map matches mote_hardware.
- arm_driver (node, `pixi run arm`): single bus owner. Publishes
  /joint_states for the arm, accepts soft-clamped goals on arm/goal, exposes
  arm/set_torque. Starts LIMP and goes limp on shutdown — nothing moves
  without an explicit command.
- jog (CLI, `pixi run arm-jog`): interactive per-joint jog; a client of the
  driver (no bus contention), clamped both sides, torque-off on exit.
- arm_check (`pixi run arm-check`): standalone enumeration/health + a
  ready-to-paste udev line + --save-home calibration snapshot.

Supporting changes:
- robot.yaml: `arm:` section (port, baud, IDs, per-joint soft limits, home,
  invert) — the single source of truth; limits are conservative placeholders
  to calibrate at the bench.
- mote.urdf.xacro: arm links/joints behind arm:=true (sim passes arm:=false)
  so robot_state_publisher animates the arm in TF from /joint_states.
- 99-mote.rules: commented /dev/mote_arm rule (pin by serial; arm_check
  prints the line).
- pixi.toml: feetech-servo-sdk dep; arm / arm-jog / arm-check tasks;
  mote_arm added to the test set.

Torque policy and calibration in mote_arm/README.md; human bench runbook in
mote_arm/BENCH.md. GitHub #2 (camera doesn't fit with the arm) noted as an
unresolved mechanical clash, not addressed here.

Verified: pixi run build, pixi run test (104 passed incl. 15 mote_arm),
pixi run lint all green; xacro generates with the arm on (real) and off (sim).

Co-Authored-By: Claude Opus 4.8 <noreply@anthropic.com>
Claude-Session: https://claude.ai/code/session_01TQqUVutHYLPLToYtiP8BSj

File: mote_description/urdf/mote.urdf.xacro (robot description, xacro)
@@ -8,4 +8,10 @@
   <xacro:arg name="sim_controllers_file" default=""/>
   <xacro:property name="use_sim" value="$(arg use_sim)"/>
+  <!-- SO-101 follower arm links. On by default (the arm is mounted); the sim
+       passes arm:=false since it does not model the arm. The joint names match
+       mote_description/config/robot.yaml and the /joint_states published by
+       mote_arm's driver, so robot_state_publisher animates the arm in TF. -->
+  <xacro:arg name="arm" default="true"/>
+  <xacro:property name="arm" value="$(arg arm)"/>
   <!-- ===================== MEASUREMENTS ===================== -->
   <!--
@@ -174,4 +180,91 @@
     <origin xyz="0 0 0" rpy="${-pi/2} 0 ${-pi/2}"/>
   </joint>
+  <!-- ===================== SO-101 FOLLOWER ARM ===================== -->
+  <!--
+    Approximate geometry for TF/visualisation only (not dynamics): each link is
+    a thin cylinder along its parent-to-child offset. Joint axes follow the
+    SO-101 kinematics (pan about Z, lift/elbow/wrist_flex about Y, roll about X).
+    Link lengths are nominal; refine if a collision model is ever needed. The
+    URDF joint limits are generous — the soft limits that actually gate motion
+    live in robot.yaml and are enforced by the mote_arm driver.
+  -->
+  <xacro:if value="${arm}">
+    <material name="arm_grey"><color rgba="0.35 0.35 0.38 1.0"/></material>
+    <xacro:macro name="arm_link" params="name length radius:=0.018">
+      <link name="${name}">
+        <visual>
+          <origin xyz="0 0 ${length/2}" rpy="0 0 0"/>
+          <geometry><cylinder radius="${radius}" length="${length}"/></geometry>
+          <material name="arm_grey"/>
+        </visual>
+      </link>
+    </xacro:macro>
+    <!-- Arm base: mounted on the top plate, roughly centred. -->
+    <link name="arm_base_link">
+      <visual>
+        <geometry><box size="0.05 0.05 0.03"/></geometry>
+        <material name="arm_grey"/>
+      </visual>
+    </link>
+    <joint name="arm_mount_joint" type="fixed">
+      <parent link="top_plate_link"/>
+      <child  link="arm_base_link"/>
+      <origin xyz="0.0 0 0.015" rpy="0 0 0"/>
+    </joint>
+    <!-- shoulder_pan: yaw about Z -->
+    <xacro:arm_link name="shoulder_pan_link" length="0.04"/>
+    <joint name="shoulder_pan" type="revolute">
+      <parent link="arm_base_link"/>
+      <child  link="shoulder_pan_link"/>
+      <origin xyz="0 0 0.015" rpy="0 0 0"/>
+      <axis xyz="0 0 1"/>
+      <limit lower="-3.14" upper="3.14" effort="10" velocity="3.0"/>
+    </joint>
+    <!-- shoulder_lift: pitch about Y (start of the upper arm) -->
+    <xacro:arm_link name="shoulder_lift_link" length="0.116"/>
+    <joint name="shoulder_lift" type="revolute">
+      <parent link="shoulder_pan_link"/>
+      <child  link="shoulder_lift_link"/>
+      <origin xyz="0 0 0.04" rpy="0 0 0"/>
+      <axis xyz="0 1 0"/>
+      <limit lower="-3.14" upper="3.14" effort="10" velocity="3.0"/>
+    </joint>
+    <!-- elbow_flex: pitch about Y -->
+    <xacro:arm_link name="elbow_flex_link" length="0.135"/>
+    <joint name="elbow_flex" type="revolute">
+      <parent link="shoulder_lift_link"/>
+      <child  link="elbow_flex_link"/>
+      <origin xyz="0 0 0.116" rpy="0 0 0"/>
+      <axis xyz="0 1 0"/>
+      <limit lower="-3.14" upper="3.14" effort="10" velocity="3.0"/>
+    </joint>
+    <!-- wrist_flex: pitch about Y -->
+    <xacro:arm_link name="wrist_flex_link" length="0.05"/>
+    <joint name="wrist_flex" type="revolute">
+      <parent link="elbow_flex_link"/>
+      <child  link="wrist_flex_link"/>
+      <origin xyz="0 0 0.135" rpy="0 0 0"/>
+      <axis xyz="0 1 0"/>
+      <limit lower="-3.14" upper="3.14" effort="10" velocity="3.0"/>
+    </joint>
+    <!-- wrist_roll: roll about X -->
+    <xacro:arm_link name="wrist_roll_link" length="0.04"/>
+    <joint name="wrist_roll" type="revolute">
+      <parent link="wrist_flex_link"/>
+      <child  link="wrist_roll_link"/>
+      <origin xyz="0 0 0.05" rpy="0 0 0"/>
+      <axis xyz="0 0 1"/>
+      <limit lower="-3.14" upper="3.14" effort="10" velocity="3.0"/>
+    </joint>
+    <!-- gripper: one actuated jaw, modelled as a revolute finger -->
+    <xacro:arm_link name="gripper_link" length="0.05" radius="0.012"/>
+    <joint name="gripper" type="revolute">
+      <parent link="wrist_roll_link"/>
+      <child  link="gripper_link"/>
+      <origin xyz="0.0 0 0.04" rpy="0 0 0"/>
+      <axis xyz="0 1 0"/>
+      <limit lower="-0.2" upper="1.7" effort="10" velocity="3.0"/>
+    </joint>
+  </xacro:if>
   <!-- ===================== ROS2 CONTROL ===================== -->
   <ros2_control name="mote_hardware" type="system">

Commit message: Benchmark: score dead-reckoning separately, and add a wheel-friction knob
Two additions to the sim benchmark harness, both useful independently of what
prompted them.

Odometry ATE: record.py now samples the odom->base pose alongside map->base, and
metrics.py reports its ATE against ground truth as `odometry.*`. The existing
localization ATE goes through AMCL's map correction, which masks changes in the
odometry underneath it; this isolates odometry quality on its own, which is what
you want when tuning kinematic_icp or sweeping localization params. report.py
surfaces it in both the aggregate and per-trial tables.

Wheel friction: a `wheel_mu` xacro arg (default 1.0, gz's own default) sets
drive-wheel friction under the existing use_sim guard, threaded through
sim_launch.py. bench.py gains --wheel-mu and a --slip shorthand (0.4). With
velocity-controlled wheels, low traction makes them spin past the ground, so the
encoders over-report motion the body never made.

Note in the README that --slip does *not* move the pose metrics much:
kinematic_icp re-registers against the scan every frame, so the slip is largely
absent from the resulting pose. It is useful for exercising code that reads the
disagreement between wheel odom and the scan-matched pose, which slip does affect.

The real-robot description is unchanged: xacro use_sim:=false output is identical
to before this commit.

Co-Authored-By: Claude Opus 4.8 <noreply@anthropic.com>
Claude-Session: https://claude.ai/code/session_01Sf64pFjR1yxSSx94jFwymB

File: mote_description/urdf/mote.urdf.xacro (robot description, xacro)
@@ -14,4 +14,9 @@
   <xacro:arg name="arm" default="true"/>
   <xacro:property name="arm" value="$(arg arm)"/>
+  <!-- Wheel-ground friction (Gazebo only). Default 1.0 reproduces gz's own
+       default surface friction; lowering it makes the velocity-controlled
+       wheels slip, so wheel odometry over-reads while the true pose lags. -->
+  <xacro:arg name="wheel_mu" default="1.0"/>
+  <xacro:property name="wheel_mu" value="$(arg wheel_mu)"/>
   <!-- ===================== MEASUREMENTS ===================== -->
   <!--
@@ -328,4 +333,13 @@
       <mu2>0.0</mu2>
     </gazebo>
+    <!-- Drive-wheel friction; wheel_mu defaults to 1.0 (gz default) -->
+    <gazebo reference="left_wheel_link">
+      <mu1>${wheel_mu}</mu1>
+      <mu2>${wheel_mu}</mu2>
+    </gazebo>
+    <gazebo reference="right_wheel_link">
+      <mu1>${wheel_mu}</mu1>
+      <mu2>${wheel_mu}</mu2>
+    </gazebo>
     <xacro:property name="lidar_sim" value="${cfg['lidar']['sim']}"/>
     <gazebo reference="lidar_link">
