Commit message: Fold SO-101 arm control into mote_hardware's ros2_control interface
The arm servos share /dev/mote_servos with the drive wheels, and a serial
port has no kernel-level exclusion, so two openers interleave packets on the
bus that moves the robot. Task 163 made that conflict safe with a port guard;
it did not make it solvable — the arm driver could not run while the base was
up, which blocked the only thing the arm is for: moving during a mission.

MoteHardware now owns the bus outright. It exports velocity command
interfaces for the wheels and position command interfaces for the six arm
joints from one open(), and arm_controller (a JointTrajectoryController) is
spawned inactive: claiming its command interfaces is what enables servo
torque, so "limp until asked" falls out of the control stack instead of being
a rule a driver has to remember.

Bus budget is why the arm is not simply read and written like the wheels.
Arm state is read one joint per cycle round-robin (~8 Hz per joint at 50 Hz)
and arm goals go out as one sync-write packet only when a goal changed, so
the arm costs about one extra transaction per cycle and nothing when idle.

The soft limits move into the hardware, on the far side of every client, so a
trajectory controller, the jog CLI and the task layer are all held to the
same envelope. Their values are unchanged.

arm_driver is retired; jog and arm_pose now command arm_controller through a
shared mote_arm.control, and never touch the bus. arm_check and arm_gains
still open it directly and still need the stack stopped.

Verified without hardware: test_arm_bus.cpp drives the real plugin through
the real SCServo SDK against a simulated STS bus on a pty and asserts on the
packets; pixi run test is green (465); pixi run sim-test passes.

File: mote_description/urdf/mote.urdf.xacro (robot description, xacro)
@@ -273,4 +273,34 @@
   </xacro:if>
   <!-- ===================== ROS2 CONTROL ===================== -->
+  <!--
+    The arm servos are on the *same* Feetech bus as the drive wheels, and a
+    serial port has no kernel-level exclusion, so one process must own it.
+    That process is the controller_manager: MoteHardware exports velocity
+    interfaces for the wheels and position interfaces for the arm, and the arm
+    can therefore move during a mission with Nav2 live.
+    If the arm is ever moved onto its own bus, `arm.port != servos.port` drops
+    the arm out of this component — it would then need a hardware component of
+    its own, which is a deliberate design change rather than a config tweak.
+  -->
+  <xacro:property name="arm_on_wheel_bus"
+                  value="${arm and cfg['arm']['port'] == cfg['servos']['port']}"/>
+  <xacro:macro name="arm_control_joint" params="spec">
+    <joint name="${spec['name']}">
+      <param name="id">${spec['id']}</param>
+      <param name="min">${spec['min']}</param>
+      <param name="max">${spec['max']}</param>
+      <param name="home">${spec['home']}</param>
+      <param name="invert">${'true' if 'invert' in spec and spec['invert'] else 'false'}</param>
+      <command_interface name="position"/>
+      <state_interface   name="position"/>
+    </joint>
+  </xacro:macro>
+  <!-- xacro has no loop; recursion over the tail is the idiom. -->
+  <xacro:macro name="arm_control_joints" params="specs">
+    <xacro:if value="${len(specs) > 0}">
+      <xacro:arm_control_joint spec="${specs[0]}"/>
+      <xacro:arm_control_joints specs="${specs[1:]}"/>
+    </xacro:if>
+  </xacro:macro>
   <ros2_control name="mote_hardware" type="system">
     <xacro:unless value="${use_sim}">
@@ -283,4 +313,8 @@
       <param name="velocity_scale">${cfg['servos']['velocity_scale']}</param>
       <param name="acceleration">${cfg['servos']['acceleration']}</param>
+      <xacro:if value="${arm_on_wheel_bus}">
+      <param name="arm_moving_speed">${cfg['arm']['moving_speed']}</param>
+      <param name="arm_moving_acc">${cfg['arm']['moving_acc']}</param>
+      </xacro:if>
     </hardware>
     </xacro:unless>
@@ -300,4 +334,17 @@
       <state_interface   name="position"/>
     </joint>
+    <!--
+      Arm joints. The bus ID, soft limits, zero offset and direction ride on
+      the joint itself rather than in the <hardware> block, so robot.yaml stays
+      the single source of truth and MoteHardware never has to reconstruct
+      which parameter belongs to which joint. The soft limits here are the
+      authoritative gate on motion: every client (a trajectory controller, the
+      jog CLI, the task layer) is clamped by the hardware, not by itself.
+      The sim runs with arm:=false — gz_ros2_control would need matching SDF
+      joints, and the sim does not model the arm.
+    -->
+    <xacro:if value="${arm_on_wheel_bus}">
+    <xacro:arm_control_joints specs="${cfg['arm']['joints']}"/>
+    </xacro:if>
   </ros2_control>
   <xacro:if value="${use_sim}">

Commit message: Resolve the arm calibration into the URDF, so the hardware clamps the right arm
Rebase onto #71, which moved this arm's zero/min/max out of the packaged
robot.yaml and into per-robot $MOTE_HOME/arm.yaml, and renamed `home:` to
`zero:` to stop it colliding with the taught rest pose.

That broke the fold semantically, not just textually. MoteHardware enforces
the soft limits and reads them from <ros2_control> params, and the xacro read
robot.yaml directly — so a calibrated robot would have been clamped against
the packaged placeholders. Those are not merely wider or narrower: calibration
moves the zero, so the same radian value names a different physical position,
and shoulder_pan's placeholder band does not contain its own zero at all.

launch_utils.resolved_arm now overlays the two through mote_arm.config.load —
the one implementation of that overlay — and hands the result to xacro as
`arm_config:=`. A bare `xacro mote.urdf.xacro` still falls back to the packaged
defaults for checking generation, and says why it must not be driven from.

Resolving at launch means the base launch needs mote_arm.config, so
arm_launch.py moves from mote_arm into mote_bringup and the dependency runs
mote_bringup -> mote_arm only; `pixi run arm` follows it. ArmJoint's
home_counts becomes zero_counts to match the vocabulary #71 established, and
records that if the homing offset turns out to apply to commanded goals it
must be compensated on both sides of the language boundary, never one.

test_the_urdf_gets_the_calibrated_zero_and_limits writes a calibration with
the real writer and asserts it reaches the emitted URDF. 607 tests green,
sim-test passes.

File: mote_description/urdf/mote.urdf.xacro (robot description, xacro)
@@ -283,6 +283,22 @@
     its own, which is a deliberate design change rather than a config tweak.
   -->
+  <!--
+    Which arm to describe. `zero`, `min` and `max` are measurements of one
+    physical arm, so a calibrated robot keeps them in $MOTE_HOME/arm.yaml, not
+    here (see robot.yaml's arm section and `pixi run arm-calibrate`). The launch
+    files resolve packaged defaults against that file and pass the result as
+    `arm_config`, which is what puts the *calibrated* limits into <ros2_control>
+    — and so into the clamp MoteHardware enforces on every client.
+    Left empty (a bare `xacro mote.urdf.xacro`, for checking generation) it
+    falls back to robot.yaml's own arm section: the conservative placeholders
+    documented there. Never drive a calibrated arm from that URDF — its zeros
+    name different physical positions.
+  -->
+  <xacro:arg name="arm_config" default=""/>
+  <xacro:property name="arm_config_file" value="$(arg arm_config)"/>
+  <xacro:property name="arm_cfg"
+                  value="${xacro.load_yaml(arm_config_file) if arm_config_file else cfg['arm']}"/>
   <xacro:property name="arm_on_wheel_bus"
-                  value="${arm and cfg['arm']['port'] == cfg['servos']['port']}"/>
+                  value="${arm and arm_cfg['port'] == cfg['servos']['port']}"/>
   <xacro:macro name="arm_control_joint" params="spec">
     <joint name="${spec['name']}">
@@ -290,5 +306,7 @@
       <param name="min">${spec['min']}</param>
       <param name="max">${spec['max']}</param>
-      <param name="home">${spec['home']}</param>
+      <!-- The encoder count reading 0 rad. Deliberately not "home": home is a
+           taught rest pose in arm_poses.yaml, a different place entirely. -->
+      <param name="zero">${spec['zero']}</param>
       <param name="invert">${'true' if 'invert' in spec and spec['invert'] else 'false'}</param>
       <command_interface name="position"/>
@@ -314,6 +332,6 @@
       <param name="acceleration">${cfg['servos']['acceleration']}</param>
       <xacro:if value="${arm_on_wheel_bus}">
-      <param name="arm_moving_speed">${cfg['arm']['moving_speed']}</param>
-      <param name="arm_moving_acc">${cfg['arm']['moving_acc']}</param>
+      <param name="arm_moving_speed">${arm_cfg['moving_speed']}</param>
+      <param name="arm_moving_acc">${arm_cfg['moving_acc']}</param>
       </xacro:if>
     </hardware>
@@ -345,5 +363,5 @@
     -->
     <xacro:if value="${arm_on_wheel_bus}">
-    <xacro:arm_control_joints specs="${cfg['arm']['joints']}"/>
+    <xacro:arm_control_joints specs="${arm_cfg['joints']}"/>
     </xacro:if>
   </ros2_control>

Commit message: Fold SO-101 arm control into mote_hardware ros2_control (single owner of the shared servo bus) (#74)
* Fold SO-101 arm control into mote_hardware's ros2_control interface

The arm servos share /dev/mote_servos with the drive wheels, and a serial
port has no kernel-level exclusion, so two openers interleave packets on the
bus that moves the robot. Task 163 made that conflict safe with a port guard;
it did not make it solvable — the arm driver could not run while the base was
up, which blocked the only thing the arm is for: moving during a mission.

MoteHardware now owns the bus outright. It exports velocity command
interfaces for the wheels and position command interfaces for the six arm
joints from one open(), and arm_controller (a JointTrajectoryController) is
spawned inactive: claiming its command interfaces is what enables servo
torque, so "limp until asked" falls out of the control stack instead of being
a rule a driver has to remember.

Bus budget is why the arm is not simply read and written like the wheels.
Arm state is read one joint per cycle round-robin (~8 Hz per joint at 50 Hz)
and arm goals go out as one sync-write packet only when a goal changed, so
the arm costs about one extra transaction per cycle and nothing when idle.

The soft limits move into the hardware, on the far side of every client, so a
trajectory controller, the jog CLI and the task layer are all held to the
same envelope. Their values are unchanged.

arm_driver is retired; jog and arm_pose now command arm_controller through a
shared mote_arm.control, and never touch the bus. arm_check and arm_gains
still open it directly and still need the stack stopped.

Verified without hardware: test_arm_bus.cpp drives the real plugin through
the real SCServo SDK against a simulated STS bus on a pty and asserts on the
packets; pixi run test is green (465); pixi run sim-test passes.

* Resolve the arm calibration into the URDF, so the hardware clamps the right arm

Rebase onto #71, which moved this arm's zero/min/max out of the packaged
robot.yaml and into per-robot $MOTE_HOME/arm.yaml, and renamed `home:` to
`zero:` to stop it colliding with the taught rest pose.

That broke the fold semantically, not just textually. MoteHardware enforces
the soft limits and reads them from <ros2_control> params, and the xacro read
robot.yaml directly — so a calibrated robot would have been clamped against
the packaged placeholders. Those are not merely wider or narrower: calibration
moves the zero, so the same radian value names a different physical position,
and shoulder_pan's placeholder band does not contain its own zero at all.

launch_utils.resolved_arm now overlays the two through mote_arm.config.load —
the one implementation of that overlay — and hands the result to xacro as
`arm_config:=`. A bare `xacro mote.urdf.xacro` still falls back to the packaged
defaults for checking generation, and says why it must not be driven from.

Resolving at launch means the base launch needs mote_arm.config, so
arm_launch.py moves from mote_arm into mote_bringup and the dependency runs
mote_bringup -> mote_arm only; `pixi run arm` follows it. ArmJoint's
home_counts becomes zero_counts to match the vocabulary #71 established, and
records that if the homing offset turns out to apply to commanded goals it
must be compensated on both sides of the language boundary, never one.

test_the_urdf_gets_the_calibrated_zero_and_limits writes a calibration with
the real writer and asserts it reaches the emitted URDF. 607 tests green,
sim-test passes.

* Skip arm servos that never answered, so an unfitted arm costs no bus time

The arm is an optional extra, and the round-robin state read did not know it.
It walked every declared arm joint regardless of whether a servo had answered
at activation, and a read to a servo that is not there does not fail fast — it
costs a full serial timeout, inside the 50 Hz loop that also drives the wheels.
On a Mote built without an arm that was paid every cycle; with one dead servo,
every sixth.

Reads now skip joints whose servo never answered. That is deliberately a
different test from the one gating commands: a servo that answered but could
not be confirmed in position mode is still read, because its state still
reaches /joint_states, which is what the activation warning promises. Hence
arm_present_ alongside arm_controllable_.

Three tests pin the pair, using a simulator that can now refuse an EEPROM mode
write: an unfitted arm issues no arm reads at all while the wheels are read as
usual; a joint excluded from control is still read; and it is never commanded,
because in wheel mode a position goal is obeyed as a speed.

Note this only fixes the cost of an absent arm. Declaring that a robot has no
arm is still unwired: mote_launch.py never passes the URDF's `arm:=` argument,
so an armless robot still gets six phantom joints in /joint_states, an arm in
TF, and an arm_controller that can never activate.

File: mote_description/urdf/mote.urdf.xacro (robot description, xacro)
@@ -273,4 +273,52 @@
   </xacro:if>
   <!-- ===================== ROS2 CONTROL ===================== -->
+  <!--
+    The arm servos are on the *same* Feetech bus as the drive wheels, and a
+    serial port has no kernel-level exclusion, so one process must own it.
+    That process is the controller_manager: MoteHardware exports velocity
+    interfaces for the wheels and position interfaces for the arm, and the arm
+    can therefore move during a mission with Nav2 live.
+    If the arm is ever moved onto its own bus, `arm.port != servos.port` drops
+    the arm out of this component — it would then need a hardware component of
+    its own, which is a deliberate design change rather than a config tweak.
+  -->
+  <!--
+    Which arm to describe. `zero`, `min` and `max` are measurements of one
+    physical arm, so a calibrated robot keeps them in $MOTE_HOME/arm.yaml, not
+    here (see robot.yaml's arm section and `pixi run arm-calibrate`). The launch
+    files resolve packaged defaults against that file and pass the result as
+    `arm_config`, which is what puts the *calibrated* limits into <ros2_control>
+    — and so into the clamp MoteHardware enforces on every client.
+    Left empty (a bare `xacro mote.urdf.xacro`, for checking generation) it
+    falls back to robot.yaml's own arm section: the conservative placeholders
+    documented there. Never drive a calibrated arm from that URDF — its zeros
+    name different physical positions.
+  -->
+  <xacro:arg name="arm_config" default=""/>
+  <xacro:property name="arm_config_file" value="$(arg arm_config)"/>
+  <xacro:property name="arm_cfg"
+                  value="${xacro.load_yaml(arm_config_file) if arm_config_file else cfg['arm']}"/>
+  <xacro:property name="arm_on_wheel_bus"
+                  value="${arm and arm_cfg['port'] == cfg['servos']['port']}"/>
+  <xacro:macro name="arm_control_joint" params="spec">
+    <joint name="${spec['name']}">
+      <param name="id">${spec['id']}</param>
+      <param name="min">${spec['min']}</param>
+      <param name="max">${spec['max']}</param>
+      <!-- The encoder count reading 0 rad. Deliberately not "home": home is a
+           taught rest pose in arm_poses.yaml, a different place entirely. -->
+      <param name="zero">${spec['zero']}</param>
+      <param name="invert">${'true' if 'invert' in spec and spec['invert'] else 'false'}</param>
+      <command_interface name="position"/>
+      <state_interface   name="position"/>
+    </joint>
+  </xacro:macro>
+  <!-- xacro has no loop; recursion over the tail is the idiom. -->
+  <xacro:macro name="arm_control_joints" params="specs">
+    <xacro:if value="${len(specs) > 0}">
+      <xacro:arm_control_joint spec="${specs[0]}"/>
+      <xacro:arm_control_joints specs="${specs[1:]}"/>
+    </xacro:if>
+  </xacro:macro>
   <ros2_control name="mote_hardware" type="system">
     <xacro:unless value="${use_sim}">
@@ -283,4 +331,8 @@
       <param name="velocity_scale">${cfg['servos']['velocity_scale']}</param>
       <param name="acceleration">${cfg['servos']['acceleration']}</param>
+      <xacro:if value="${arm_on_wheel_bus}">
+      <param name="arm_moving_speed">${arm_cfg['moving_speed']}</param>
+      <param name="arm_moving_acc">${arm_cfg['moving_acc']}</param>
+      </xacro:if>
     </hardware>
     </xacro:unless>
@@ -300,4 +352,17 @@
       <state_interface   name="position"/>
     </joint>
+    <!--
+      Arm joints. The bus ID, soft limits, zero offset and direction ride on
+      the joint itself rather than in the <hardware> block, so robot.yaml stays
+      the single source of truth and MoteHardware never has to reconstruct
+      which parameter belongs to which joint. The soft limits here are the
+      authoritative gate on motion: every client (a trajectory controller, the
+      jog CLI, the task layer) is clamped by the hardware, not by itself.
+      The sim runs with arm:=false — gz_ros2_control would need matching SDF
+      joints, and the sim does not model the arm.
+    -->
+    <xacro:if value="${arm_on_wheel_bus}">
+    <xacro:arm_control_joints specs="${arm_cfg['joints']}"/>
+    </xacro:if>
   </ros2_control>
   <xacro:if value="${use_sim}">
